File: new.kicad_pcb (KiCad board)
At the start: 2 copper layers, 55.9 x 91.4 mm, 4 parts, among them P1 CONN_02X16, P2 CONN_02X16, P3 CONN_01X32, P4 CONN_01X32

Commit message: small changes
Parts:
- moved P3 68.4 mm to (33.8, 20.3)
- moved P1 68.4 mm to (65.1, 40.6)
- moved P4 68.4 mm to (49.0, 20.3)
- moved P2 67.5 mm to (20.3, 40.6)
Routing:
- net /33: track 23.9 -> 28.0 mm
- net /35: track 22.1 -> 25.6 mm
- net /60: track 26.6 -> 23.5 mm
- net /36: track 23.2 -> 26.2 mm
- net /37: track 18.8 -> 21.6 mm
- net /61: track 23.7 -> 20.9 mm
- net /63: track 25.9 -> 23.4 mm
- net /57: track 20.0 -> 17.7 mm
- net /34: track 26.3 -> 28.6 mm
- net /59: track 21.5 -> 19.3 mm
- net /38: track 21.4 -> 23.3 mm
- net /62: track 28.8 -> 27.0 mm
- net /64: track 29.6 -> 27.8 mm
- net /58: track 23.7 -> 22.2 mm
- net /39: track 17.7 -> 19.0 mm
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Other:
- board text added: "QFP64-ADAPTER-V1"

Commit message: changed the pad's shape and added copper pour layer
Routing:
- net (no net): track 4.62 -> 0.43 mm
- added copper zone on B.Cu, net (none)
- added copper zone on F.Cu, net (none)
Changed lines of the file:
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@@
     (area 13.132999 13.894999 69.163001 105.485001)
     (thickness 1.6)
-    (drawings 13)
-    (tracks 365)
+    (drawings 15)
+    (tracks 361)
     (zones 0)
     (modules 4)
@@
   (page A4)
   (layers
-    (0 F.Cu signal)
-    (31 B.Cu signal)
+    (0 F.Cu signal hide)
+    (31 B.Cu signal hide)
     (32 B.Adhes user hide)
     (33 F.Adhes user hide)
@@
     (35 F.Paste user hide)
     (36 B.SilkS user hide)
-    (37 F.SilkS user hide)
+    (37 F.SilkS user)
     (38 B.Mask user hide)
     (39 F.Mask user hide)
@@
       (effects (font (size 1 1) (thickness 0.15)))
     )
-    (pad 1 thru_hole rect (at 0 0) (size 1.7 1.7) (drill 1) (layers *.Cu *.Mask)
+    (pad 1 thru_hole circle (at 0 0) (size 1.7 1.7) (drill 1) (layers *.Cu *.Mask)
       (net 33 /33))
     (pad 2 thru_hole oval (at -2.54 0) (size 1.7 1.7) (drill 1) (layers *.Cu *.Mask)
@@
     )
   )
+  (gr_line (start 65.024 37.846) (end 64.77 37.592) (angle 90) (layer F.SilkS) (width 0.2))
+  (gr_line (start 65.278 37.592) (end 65.024 37.846) (angle 90) (layer F.SilkS) (width 0.2))
+  (gr_line (start 64.77 37.592) (end 65.278 37.592) (angle 90) (layer F.SilkS) (width 0.2))
   (gr_text QFP64-ADAPTER-V1 (at 25.4 103.632) (layer B.Cu)
     (effects (font (size 1.5 1.5) (thickness 0.3)) (justify mirror))
@@
     (effects (font (size 1.5 1.5) (thickness 0.3)))
   )
-  (gr_circle (center 68.072 40.386) (end 68.326 40.894) (layer F.SilkS) (width 0.2))
   (gr_text "51\n52\n53\n54\n55\n56\n57\n58\n59\n60\n61\n62\n63\n64" (at 30.48 82.55) (layer F.SilkS)
     (effects (font (size 1.5 1.5) (thickness 0.3)))
@@
   (gr_line (start 69.088 13.97) (end 69.088 105.41) (angle 90) (layer Edge.Cuts) (width 0.15))
   (gr_line (start 13.208 13.97) (end 69.088 13.97) (angle 90) (layer Edge.Cuts) (width 0.15))
-  (segment (start 67.564 40.386) (end 68.326 39.624) (width 0.25) (layer B.Cu) (net 0))
-  (segment (start 67.564 40.64) (end 67.564 40.386) (width 0.25) (layer B.Cu) (net 0))
-  (segment (start 68.326 41.402) (end 67.564 40.64) (width 0.25) (layer B.Cu) (net 0))
-  (segment (start 68.326 39.624) (end 68.326 41.402) (width 0.25) (layer B.Cu) (net 0))
   (segment (start 17.732 38.09) (end 17.732 38.306) (width 0.25) (layer B.Cu) (net 0))
   (segment (start 17.732 38.09) (end 17.732 38.306) (width 0.25) (layer B.Cu) (net 0))
@@
   (segment (start 18.581999 79.539999) (end 18.581999 79.541999) (width 0.25) (layer B.Cu) (net 64))
   (segment (start 33.782 99.06) (end 33.782 98.298) (width 0.25) (layer B.Cu) (net 64))
+  (zone (net 0) (net_name "") (layer F.Cu) (hatch edge 0.508)
+    (connect_pads (clearance 0.508))
+    (min_thickness 0.254)
+    (fill yes (arc_segments 16) (thermal_gap 0.508) (thermal_bridge_width 0.508))
+    (polygon
+      (pts
+        (xy 69.088 105.41) (xy 13.208 105.41) (xy 13.208 13.97) (xy 69.088 13.97)
+      )
+    )
+  )
+  (zone (net 0) (net_name "") (layer B.Cu) (hatch edge 0.508)
+    (connect_pads (clearance 0.508))
+    (min_thickness 0.254)
+    (fill yes (arc_segments 16) (thermal_gap 0.508) (thermal_bridge_width 0.508))
+    (polygon
+      (pts
+        (xy 69.088 105.41) (xy 13.208 105.41) (xy 13.208 13.97) (xy 69.088 13.97)
+      )
+    )
+  )
 )
